File: hardware/PowerShift.kicad_pcb (KiCad board)
At the start: 2 copper layers, 50 x 90 mm, 62 parts, among them J1 Barrel_Jack, J10 SHIFT_IN, J11 JST-ZR, J12 JST-ZR, J14 JST-ZR, J2 MICRO_USB, J3 JST-ZR, J4 JST-ZR, J5 SHIFT_IN, J6 SHIFT_IN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

Commit message: Nearly there
Routing:
- net GND: track 234.5 -> 301.5 mm, vias 42 -> 65
- net /SER_OUT: track 0.00 -> 54.8 mm
- net VPP: track 69.1 -> 122.0 mm, vias 6 -> 9
- net /RCK: track 114.7 -> 151.4 mm, vias 2 -> 7
- net /~G: track 118.9 -> 154.7 mm, vias 2 -> 3
- net /SER_IN: track 56.3 -> 90.4 mm, vias 2 -> 3
- net +3V3: track 265.5 -> 293.4 mm
- net /SRCK: track 126.1 -> 146.6 mm, vias 10 -> 13
- net /~SRCLR: track 126.1 -> 132.8 mm
- net Net-(J5-Pad8): track 0.00 -> 3.40 mm
- net Net-(J5-Pad2): track 0.00 -> 3.25 mm

Commit message: All nets connected, DRC OK
Routing:
- net GND: track 301.5 -> 322.4 mm, vias 65 -> 68
- net /~SRCLR: track 132.8 -> 149.4 mm
- net /SRCK: track 146.6 -> 162.0 mm, vias 13 -> 14
Changed lines of the file:
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@@
   (general
     (links 227)
-    (no_connects 4)
+    (no_connects 0)
     (area 20.435716 39.974999 106.325001 162.700001)
     (thickness 1.6)
     (drawings 10)
-    (tracks 1084)
+    (tracks 1115)
     (zones 0)
     (modules 62)
@@
   )
   (setup
-    (last_trace_width 0.5)
+    (last_trace_width 0.25)
     (user_trace_width 0.5)
     (user_trace_width 0.75)
@@
   (segment (start 71.625 79.125) (end 75.5 75.25) (width 1) (layer B.Cu) (net 1))
   (segment (start 75.5 75.25) (end 75.5 75.14) (width 1) (layer B.Cu) (net 1))
+  (segment (start 86.3 54.66) (end 87.1025 54.66) (width 0.25) (layer B.Cu) (net 2))
+  (segment (start 87.1025 54.66) (end 87.4625 54.3) (width 0.25) (layer B.Cu) (net 2))
+  (segment (start 86.75 101) (end 86.75 103.5) (width 0.5) (layer B.Cu) (net 2))
+  (segment (start 86.5 100.75) (end 86.75 101) (width 0.5) (layer B.Cu) (net 2))
+  (segment (start 85 100.75) (end 86.5 100.75) (width 0.5) (layer B.Cu) (net 2))
+  (segment (start 82.75 103) (end 85 100.75) (width 0.5) (layer B.Cu) (net 2))
+  (segment (start 80.75 103) (end 82.75 103) (width 0.5) (layer B.Cu) (net 2))
+  (segment (start 79.05 102.965) (end 80.715 102.965) (width 0.5) (layer F.Cu) (net 2))
+  (segment (start 80.715 102.965) (end 80.75 103) (width 0.5) (layer F.Cu) (net 2))
+  (via (at 80.75 103) (size 0.6) (drill 0.4) (layers F.Cu B.Cu) (net 2))
+  (segment (start 72.5 103) (end 70.735 103) (width 0.75) (layer F.Cu) (net 2))
+  (segment (start 70.735 103) (end 70.7 102.965) (width 0.75) (layer F.Cu) (net 2))
+  (segment (start 77.5 103) (end 72.5 103) (width 0.75) (layer B.Cu) (net 2))
+  (via (at 72.5 103) (size 0.6) (drill 0.4) (layers F.Cu B.Cu) (net 2))
+  (segment (start 79.05 102.965) (end 77.535 102.965) (width 0.75) (layer F.Cu) (net 2))
+  (segment (start 77.535 102.965) (end 77.5 103) (width 0.75) (layer F.Cu) (net 2))
+  (via (at 77.5 103) (size 0.6) (drill 0.4) (layers F.Cu B.Cu) (net 2))
   (segment (start 86.75 117.75) (end 86.75 119.5) (width 0.5) (layer B.Cu) (net 2))
   (segment (start 86.25 117.25) (end 86.75 117.75) (width 0.5) (layer B.Cu) (net 2))
@@
   (segment (start 52.25 115.13) (end 55.49 115.13) (width 0.75) (layer F.Cu) (net 32))
   (segment (start 55.49 115.13) (end 55.5 115.14) (width 0.75) (layer F.Cu) (net 32))
+  (segment (start 86.5 133) (end 88.375 133) (width 0.25) (layer F.Cu) (net 33))
+  (segment (start 88.375 133) (end 88.45 132.925) (width 0.25) (layer F.Cu) (net 33))
+  (segment (start 80.5 133.5) (end 86 133.5) (width 0.25) (layer B.Cu) (net 33))
+  (segment (start 86 133.5) (end 86.5 133) (width 0.25) (layer B.Cu) (net 33))
+  (via (at 86.5 133) (size 0.6) (drill 0.4) (layers F.Cu B.Cu) (net 33))
+  (segment (start 80.375001 133.375001) (end 80.5 133.5) (width 0.25) (layer B.Cu) (net 33))
+  (segment (start 79 132) (end 80.375001 133.375001) (width 0.25) (layer B.Cu) (net 33))
+  (segment (start 75.25 132) (end 79 132) (width 0.25) (layer B.Cu) (net 33))
+  (segment (start 74.549999 132.700001) (end 75.25 132) (width 0.25) (layer B.Cu) (net 33))
+  (segment (start 74.25 133) (end 74.549999 132.700001) (width 0.25) (layer B.Cu) (net 33))
   (segment (start 61 120.5) (end 52.54 120.5) (width 0.25) (layer B.Cu) (net 33))
   (segment (start 52.54 120.5) (end 52.25 120.21) (width 0.25) (layer B.Cu) (net 33))
@@
   (segment (start 77.055 101.695) (end 76.5 102.25) (width 0.25) (layer F.Cu) (net 35))
   (segment (start 79.05 101.695) (end 77.055 101.695) (width 0.25) (layer F.Cu) (net 35))
+  (segment (start 75.75 133) (end 75 133.75) (width 0.25) (layer B.Cu) (net 36))
+  (segment (start 75 133.75) (end 60.5 133.75) (width 0.25) (layer B.Cu) (net 36))
+  (segment (start 60.5 133.75) (end 59.75 133) (width 0.25) (layer B.Cu) (net 36))
   (segment (start 58.5 116.75) (end 58.5 126.75) (width 0.25) (layer F.Cu) (net 36))
   (segment (start 58.5 126.75) (end 58.5 132.75) (width 0.25) (layer F.Cu) (net 36))
@@
   (segment (start 81.325 94.075) (end 81.75 94.5) (width 0.25) (layer F.Cu) (net 82))
   (segment (start 79.05 94.075) (end 81.325 94.075) (width 0.25) (layer F.Cu) (net 82))
+  (segment (start 83.75 113.5) (end 83.75 104) (width 0.25) (layer B.Cu) (net 83))
+  (segment (start 85.75 102) (end 85.450001 102.299999) (width 0.25) (layer B.Cu) (net 83))
+  (segment (start 85.450001 102.299999) (end 83.75 104) (width 0.25) (layer B.Cu) (net 83))
+  (segment (start 85.75 100) (end 85.75 102) (width 0.25) (layer F.Cu) (net 83))
+  (via (at 85.75 102) (size 0.6) (drill 0.4) (layers F.Cu B.Cu) (net 83))
   (segment (start 86.175 94.075) (end 85.75 94.5) (width 0.25) (layer F.Cu) (net 83))
   (segment (start 85.75 94.5) (end 85.75 94.75) (width 0.25) (layer F.Cu) (net 83))
   (segment (start 88.45 94.075) (end 86.175 94.075) (width 0.25) (layer F.Cu) (net 83))
   (segment (start 85.75 100) (end 85.75 94.75) (width 0.25) (layer F.Cu) (net 83))
-  (segment (start 83.75 103.25) (end 83.75 102) (width 0.25) (layer B.Cu) (net 83))
-  (segment (start 83.75 102) (end 85.75 100) (width 0.25) (layer B.Cu) (net 83))
-  (via (at 85.75 100) (size 0.6) (drill 0.4) (layers F.Cu B.Cu) (net 83))
-  (segment (start 83.75 113.5) (end 83.75 103.25) (width 0.25) (layer B.Cu) (net 83))
   (segment (start 83.75 114.5) (end 83.75 113.5) (width 0.25) (layer B.Cu) (net 83))
   (segment (start 81.75 116.5) (end 83.75 114.5) (width 0.25) (layer B.Cu) (net 83))

Commit message: Silkscreen
Other:
- board text added: "C1"
- board text added: "C10"
- board text added: "C12"
- board text added: "C13"
- board text added: "C14"
- board text added: "C17"
- board text added: "C18"
- board text added: "C19"
- board text added: "C2"
- board text added: "C20"
- board text added: "C21"
- board text added: "C22"
- board text added: "C3"
- board text added: "C4"
- board text added: "C5"
- board text added: "C6"
- board text added: "C7"
- board text added: "C8"
- board text added: "D1"
- board text added: "J5"
- board text added: "JMP2"
- board text added: "JMP4"
- board text added: "R3"
- board text added: "R4"
- board text added: "R5"
- board text added: "R6"
- board text added: "U1"
- board text added: "U10"
- board text added: "U2"
- board text added: "U3"
- board text added: "U4"
- board text added: "U5"
- board text added: "U7"
- board text added: "U9"

Commit message: Top silk
Other:
- board text added: "J7"
Changed lines of the file:
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@@
     (area 20.435716 39.974999 106.325001 162.700001)
     (thickness 1.6)
-    (drawings 118)
+    (drawings 146)
     (tracks 1115)
     (zones 0)
@@
     )
   )
+  (gr_line (start 98.75 70.5) (end 98.75 69.5) (layer Eco1.User) (width 0.2))
+  (gr_line (start 97.25 69.5) (end 97.25 70.5) (layer Eco1.User) (width 0.2))
+  (gr_line (start 98.75 65) (end 98.75 66) (layer Eco1.User) (width 0.2))
+  (gr_line (start 97.25 65) (end 97.25 66) (layer Eco1.User) (width 0.2))
+  (gr_line (start 93 63.75) (end 97 63.75) (layer Eco1.User) (width 0.2))
+  (gr_line (start 93 71.75) (end 93 63.75) (layer Eco1.User) (width 0.2))
+  (gr_line (start 97 71.75) (end 93 71.75) (layer Eco1.User) (width 0.2))
+  (gr_line (start 97 63.75) (end 97 71.75) (layer Eco1.User) (width 0.2))
+  (gr_line (start 80.75 65.75) (end 80.75 64.75) (layer Eco1.User) (width 0.2))
+  (gr_line (start 79.25 64.75) (end 79.25 65.75) (layer Eco1.User) (width 0.2))
+  (gr_line (start 78.75 65.75) (end 78.75 64.75) (layer Eco1.User) (width 0.2))
+  (gr_line (start 77.25 64.75) (end 77.25 65.75) (layer Eco1.User) (width 0.2))
+  (gr_line (start 66 68.75) (end 68 68.75) (layer Eco1.User) (width 0.2))
+  (gr_line (start 66 65.25) (end 68 65.25) (layer Eco1.User) (width 0.2))
+  (gr_line (start 66 70.75) (end 67 70.75) (layer Eco1.User) (width 0.2))
+  (gr_line (start 66 69.25) (end 67 69.25) (layer Eco1.User) (width 0.2))
+  (gr_line (start 95.5 63) (end 94.5 63) (layer Eco1.User) (width 0.2))
+  (gr_line (start 94.5 61.5) (end 95.5 61.5) (layer Eco1.User) (width 0.2))
+  (gr_line (start 95.5 60.75) (end 94.5 60.75) (layer Eco1.User) (width 0.2))
+  (gr_line (start 94.5 59.25) (end 95.5 59.25) (layer Eco1.User) (width 0.2))
+  (gr_circle (center 90.5 81.75) (end 91 81.75) (layer Eco1.User) (width 0.2))
+  (gr_text J7 (at 92.25 80) (layer Eco1.User)
+    (effects (font (size 1 1) (thickness 0.15)))
+  )
+  (gr_line (start 97 81) (end 94.5 81) (layer Eco1.User) (width 0.2))
+  (gr_line (start 97 89) (end 97 81) (layer Eco1.User) (width 0.2))
+  (gr_line (start 91.5 89) (end 97 89) (layer Eco1.User) (width 0.2))
+  (gr_line (start 91.5 84) (end 91.5 89) (layer Eco1.User) (width 0.2))
+  (gr_line (start 91.5 81) (end 91.5 82.5) (layer Eco1.User) (width 0.2))
+  (gr_line (start 91.5 81) (end 93 81) (layer Eco1.User) (width 0.2))
   (gr_circle (center 96 136) (end 92.75 136) (layer Eco1.User) (width 0.2))
   (gr_circle (center 54 136) (end 57.25 136.25) (layer Eco1.User) (width 0.2))

Commit message: Buttons
Parts:
- added SW1: SW_Push, kuro:Switch_FSM-JSM-Series, F.Cu at (75.0, 72.0)
- added SW2: SW_Push, kuro:Switch_FSM-JSM-Series, F.Cu at (75.0, 86.0)
Connections:
- J7 pad 3: (no net) -> Net-(J7-Pad3)
- J7 pad 4: (no net) -> Net-(J7-Pad4)
- U10 pad 5: (no net) -> Net-(U10-Pad5)
- U2 pad 1: (no net) -> Net-(U2-Pad1)
- U2 pad 20: (no net) -> Net-(U2-Pad20)
- U3 pad 1: (no net) -> Net-(U3-Pad1)
- U3 pad 20: (no net) -> Net-(U3-Pad20)
- U4 pad 1: (no net) -> Net-(U4-Pad1)
- U4 pad 20: (no net) -> Net-(U4-Pad20)
- U5 pad 1: (no net) -> Net-(U5-Pad1)
- U5 pad 20: (no net) -> Net-(U5-Pad20)
- U7 pad 1: (no net) -> Net-(U7-Pad1)
- U7 pad 20: (no net) -> Net-(U7-Pad20)
- U8 pad 1: (no net) -> Net-(U8-Pad1)
- U8 pad 20: (no net) -> Net-(U8-Pad20)
- U9 pad 10: (no net) -> /BTN1
- U9 pad 12: (no net) -> Net-(U9-Pad12)
- U9 pad 13: (no net) -> /BTN2
- U9 pad 2: (no net) -> Net-(U9-Pad2)
- U9 pad 29: (no net) -> Net-(U9-Pad29)
- U9 pad 30: (no net) -> Net-(U9-Pad30)
- U9 pad 31: (no net) -> Net-(U9-Pad31)
Routing:
- net /BTN2: track 0.00 -> 39.6 mm, vias 0 -> 2
- net GND: track 322.4 -> 339.7 mm
- net /BTN1: track 0.00 -> 16.9 mm, vias 0 -> 2
Other:
- board text added: "SW1"
- board text added: "SW2"

Commit message: Corrected top silk for buttons
Other:
- board text added: "C11"
- board text added: "C15"
- board text added: "C16"
- board text added: "C9"
- board text added: "U6"
- board text added: "Y1"
Changed lines of the file:
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@@
     (area 49.924999 49.924999 100.075001 140.075001)
     (thickness 1.6)
-    (drawings 158)
+    (drawings 175)
     (tracks 1146)
     (zones 0)
@@
       (net 2 GND))
   )
+  (gr_line (start 83.75 60.75) (end 82.75 60.75) (layer Eco1.User) (width 0.2))
+  (gr_line (start 82.75 59.25) (end 83.75 59.25) (layer Eco1.User) (width 0.2))
+  (gr_text C16 (at 99.5 70 90) (layer Eco1.User)
+    (effects (font (size 1 1) (thickness 0.15)))
+  )
+  (gr_text C15 (at 99.5 65.5 90) (layer Eco1.User)
+    (effects (font (size 1 1) (thickness 0.15)))
+  )
+  (gr_text Y1 (at 95 67.75) (layer Eco1.User)
+    (effects (font (size 1 1) (thickness 0.15)))
+  )
+  (gr_line (start 93.25 72.25) (end 92.25 72.25) (layer Eco1.User) (width 0.2))
+  (gr_line (start 92.25 73.75) (end 93.25 73.75) (layer Eco1.User) (width 0.2))
+  (gr_text C11 (at 92.25 74.75) (layer Eco1.User)
+    (effects (font (size 1 1) (thickness 0.15)))
+  )
+  (gr_circle (center 99.25 76.75) (end 99.75 76.75) (layer Eco1.User) (width 0.2))
+  (gr_line (start 95.25 72.25) (end 95.25 76.75) (layer Eco1.User) (width 0.2))
+  (gr_line (start 98.75 72.25) (end 95.25 72.25) (layer Eco1.User) (width 0.2))
+  (gr_line (start 98.75 75.25) (end 98.75 72.25) (layer Eco1.User) (width 0.2))
+  (gr_line (start 95.25 76.75) (end 97 76.75) (layer Eco1.User) (width 0.2))
+  (gr_line (start 97.5 78.75) (end 96.5 78.75) (layer Eco1.User) (width 0.2))
+  (gr_line (start 96.5 77.25) (end 97.5 77.25) (layer Eco1.User) (width 0.2))
+  (gr_text U6 (at 94.5 75.5 90) (layer Eco1.User)
+    (effects (font (size 1 1) (thickness 0.15)))
+  )
+  (gr_text C9 (at 94 78) (layer Eco1.User)
+    (effects (font (size 1 1) (thickness 0.15)))
+  )
   (gr_text SW2 (at 75 82) (layer Eco1.User)
     (effects (font (size 1 1) (thickness 0.15)))
@@
     (effects (font (size 1 1) (thickness 0.15)))
   )
-  (gr_circle (center 70.25 68.5) (end 70.75 68.5) (layer Eco1.User) (width 0.2))
+  (gr_circle (center 70.25 68) (end 70.75 68) (layer Eco1.User) (width 0.2))
   (gr_text U10 (at 71 65) (layer Eco1.User)
     (effects (font (size 1 1) (thickness 0.15)))
   )
-  (gr_text C17 (at 70 70) (layer Eco1.User)
+  (gr_text C17 (at 66.5 71.75) (layer Eco1.User)
     (effects (font (size 1 1) (thickness 0.15)))
   )
@@
   (gr_line (start 65.75 138.5) (end 66.75 138.5) (layer Eco1.User) (width 0.2))
   (gr_line (start 65.75 137) (end 66.75 137) (layer Eco1.User) (width 0.2))
-  (gr_text U2 (at 71 89.75) (layer Eco1.User)
+  (gr_text U2 (at 61 89.75) (layer Eco1.User)
     (effects (font (size 1 1) (thickness 0.15)))
   )
@@
     (effects (font (size 1 1) (thickness 0.15)))
   )
-  (gr_text C6 (at 80.75 89) (layer Eco1.User)
+  (gr_text C6 (at 86.75 89) (layer Eco1.User)
     (effects (font (size 1 1) (thickness 0.15)))
   )

Commit message: Bottom silk
Other:
- board text added: "0-7"
- board text added: "1"
- board text added: "16-23"
- board text added: "24-31"
- board text added: "32-39"
- board text added: "40-47"
- board text added: "5"
- board text added: "8"
- board text added: "8-15"
- board text added: "J1"
- board text added: "J10"
- board text added: "J11"
- board text added: "J12"
- board text added: "J14"
- board text added: "J2"
- board text added: "J3"
- board text added: "J4"
- board text added: "J6"
- board text added: "J8"
- board text added: "J9"
- board text added: "JMP1"
- board text added: "JMP3"
- board text added: "L1"
- board text added: "R1"
- board text added: "R2"

Commit message: Top silk fix
Other:
- board text added: "PowerShift 1.0 (C) 2018 Paul Qureshi"
Changed lines of the file:
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@@
     (area 49.924999 49.924999 100.075001 140.075001)
     (thickness 1.6)
-    (drawings 280)
+    (drawings 297)
     (tracks 1146)
     (zones 0)
@@
   (page A4)
   (layers
-    (0 F.Cu signal hide)
-    (31 B.Cu signal)
+    (0 F.Cu signal)
+    (31 B.Cu signal hide)
     (32 B.Adhes user)
     (33 F.Adhes user)
@@
     (40 Dwgs.User user)
     (41 Cmts.User user)
-    (42 Eco1.User user hide)
-    (43 Eco2.User user)
+    (42 Eco1.User user)
+    (43 Eco2.User user hide)
     (44 Edge.Cuts user)
     (45 Margin user)
-    (46 B.CrtYd user)
+    (46 B.CrtYd user hide)
     (47 F.CrtYd user hide)
     (48 B.Fab user hide)
@@
     (pad_to_mask_clearance 0.2)
     (aux_axis_origin 0 0)
-    (visible_elements 7FFFBFFF)
+    (visible_elements 7FFF7FFF)
     (pcbplotparams
       (layerselection 0x00030_80000001)
@@
       (net 2 GND))
   )
+  (gr_circle (center 54.25 111.25) (end 54.75 111.25) (layer Eco1.User) (width 0.2))
+  (gr_line (start 54.75 81.25) (end 55.25 81.25) (layer Eco1.User) (width 0.2))
+  (gr_line (start 54.5 132.25) (end 54.5 127.75) (layer Eco1.User) (width 0.2))
+  (gr_line (start 56.5 132.25) (end 54.5 132.25) (layer Eco1.User) (width 0.2))
+  (gr_line (start 56.5 127.75) (end 56.5 132.25) (layer Eco1.User) (width 0.2))
+  (gr_line (start 54.5 127.75) (end 56.5 127.75) (layer Eco1.User) (width 0.2))
+  (gr_line (start 54.5 116) (end 54.5 113) (layer Eco1.User) (width 0.2))
+  (gr_line (start 56.5 116) (end 54.5 116) (layer Eco1.User) (width 0.2))
+  (gr_line (start 56.5 113) (end 56.5 116) (layer Eco1.User) (width 0.2))
+  (gr_line (start 54.5 113) (end 56.5 113) (layer Eco1.User) (width 0.2))
+  (gr_text 40-47 (at 83.75 129.75 90) (layer Eco1.User)
+    (effects (font (size 1.5 1.5) (thickness 0.3)))
+  )
+  (gr_text 32-39 (at 83.75 113.5 90) (layer Eco1.User)
+    (effects (font (size 1.5 1.5) (thickness 0.3)))
+  )
+  (gr_text 24-31 (at 83.75 97.25 90) (layer Eco1.User)
+    (effects (font (size 1.5 1.5) (thickness 0.3)))
+  )
+  (gr_text 16-23 (at 66.25 129.75 90) (layer Eco1.User)
+    (effects (font (size 1.5 1.5) (thickness 0.3)))
+  )
+  (gr_text 8-15 (at 66.25 110.25 90) (layer Eco1.User)
+    (effects (font (size 1.5 1.5) (thickness 0.3)))
+  )
+  (gr_text 0-7 (at 66 97.25 90) (layer Eco1.User)
+    (effects (font (size 1.5 1.5) (thickness 0.3)))
+  )
+  (gr_text "PowerShift 1.0\n(C) 2018 Paul Qureshi" (at 96 130 90) (layer Eco1.User)
+    (effects (font (size 1.5 1.5) (thickness 0.3)) (justify left))
+  )
   (gr_line (start 79.75 72.75) (end 77.25 72.75) (layer Eco2.User) (width 0.2))
