File: hardware/PowerShift.kicad_pcb (KiCad board)
At the start: 2 copper layers, 50 x 90 mm, 64 parts, among them J1 Barrel_Jack, J10 SHIFT_IN, J11 JST-ZR, J12 JST-ZR, J14 JST-ZR, J2 MICRO_USB, J3 JST-ZR, J4 JST-ZR, J5 SHIFT_IN, J6 SHIFT_IN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

Commit message: Top silk
Parts:
- added G***: LOGO, Keio:logo2_16x5mm, F.Cu at (96.0, 99.0)
Other:
- board text added: "3.3V RS232"
- board text added: "GPLv3"
- board text added: "PowerShift 1.0"
- board text added: "©2018 Paul Qureshi"
- board text removed: "PowerShift 1.0 (C) 2018 Paul Qureshi"

Commit message: Silk on silk layers
Other:
- board text removed: "1"
- board text removed: "5"
- board text removed: "8"
- board text removed: "C1"
- board text removed: "C10"
- board text removed: "C11"
- board text removed: "C12"
- board text removed: "C13"
- board text removed: "C14"
- board text removed: "C15"
- board text removed: "C16"
- board text removed: "C17"
- board text removed: "C18"
- board text removed: "C19"
- board text removed: "C2"
- board text removed: "C20"
- board text removed: "C21"
- board text removed: "C22"
- board text removed: "C3"
- board text removed: "C4"
- board text removed: "C5"
- board text removed: "C6"
- board text removed: "C7"
- board text removed: "C8"
- board text removed: "C9"
- board text removed: "D1"
- board text removed: "J1"
- board text removed: "J10"
- board text removed: "J11"
- board text removed: "J12"
- board text removed: "J14"
- board text removed: "J2"
- board text removed: "J3"
- board text removed: "J4"
- board text removed: "J5"
- board text removed: "J6"
- board text removed: "J7"
- board text removed: "J8"
- board text removed: "J9"
- board text removed: "JMP1"
- board text removed: "JMP2"
- board text removed: "JMP3"
- board text removed: "JMP4"
- board text removed: "L1"
- board text removed: "R1"
- board text removed: "R2"
- board text removed: "R3"
- board text removed: "R4"
- board text removed: "R5"
- board text removed: "R6"
- board text removed: "SW1"
- board text removed: "SW2"
- board text removed: "U1"
- board text removed: "U10"
- board text removed: "U2"
- board text removed: "U3"
- board text removed: "U4"
- board text removed: "U5"
- board text removed: "U6"
- board text removed: "U7"
- board text removed: "U9"
- board text removed: "Y1"

Commit message: Keio logo on silk layer
Parts:
- G***: footprint Keio:logo2_16x5mm -> Keio:logo2_16x5mm_top_silk
Changed lines of the file:
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@@
     (links 235)
     (no_connects 0)
-    (area 49.924999 49.924999 100.075001 140.075001)
+    (area 21.150001 39.974999 106.325001 162.700001)
     (thickness 1.6)
     (drawings 67)
@@
       (net 6 "Net-(C16-Pad1)"))
   )
-  (module Keio:logo2_16x5mm (layer F.Cu)
+  (module Keio:logo2_16x5mm_top_silk (layer F.Cu)
     (at 96 99 90)
     (fp_text reference G*** (at 0 0 90) (layer F.SilkS) hide
@@
       (xy -1.09542 -2.462189) (xy -0.959649 -2.462265) (xy -0.816598 -2.462339) (xy -0.666074 -2.462412)
       (xy -0.507882 -2.462486) (xy -0.341829 -2.462559) (xy -0.16772 -2.462634) (xy 0.014638 -2.462711)
-      (xy 0.037065 -2.46272) (xy 2.79828 -2.463863) (xy 2.797199 -2.094474)) (layer Eco1.User) (width 0.01))
+      (xy 0.037065 -2.46272) (xy 2.79828 -2.463863) (xy 2.797199 -2.094474)) (layer F.SilkS) (width 0.01))
     (fp_poly (pts (xy 8.21582 -0.44349) (xy 8.215728 -0.28711) (xy 8.215639 -0.138969) (xy 8.21555 0.001161)
       (xy 8.215462 0.133508) (xy 8.215372 0.2583) (xy 8.215281 0.375764) (xy 8.215187 0.486129)
@@
       (xy 3.678846 -2.26339) (xy 3.739001 -2.305467) (xy 3.804166 -2.34366) (xy 3.830179 -2.357222)
       (xy 3.887097 -2.3841) (xy 3.943121 -2.406423) (xy 4.000647 -2.424979) (xy 4.062071 -2.440553)
-      (xy 4.119034 -2.452014) (xy 4.171951 -2.461613) (xy 8.216987 -2.463895) (xy 8.21582 -0.44349)) (layer Eco1.User) (width 0.01))
+      (xy 4.119034 -2.452014) (xy 4.171951 -2.461613) (xy 8.216987 -2.463895) (xy 8.21582 -0.44349)) (layer F.SilkS) (width 0.01))
   )
   (gr_line (start 64 140) (end 90 140) (layer Edge.Cuts) (width 0.15))
